File: staj/staj.sch (KiCad schematic (older format))
At the start: 20 parts, among them J1 Conn_01x08, J2 Conn_01x02, J3 Conn_01x02, J4 Conn_01x08, U1 AD820, U2 AD820

Commit message: Devre çizildi, projenin test devresi tamamlandı.
Parts:
- removed R12: 82.5k, symbol Device:R
- removed R13: 10k, symbol Device:R
- added 1K1, 1K2, 1K3: R, Resistor_SMD:R_0805_2012Metric, symbol Device:R
- added C1, C2: 470nF, Capacitor_SMD:C_0805_2012Metric, symbol Device:C
- added C3, C8: 10nF, Capacitor_SMD:C_0805_2012Metric, symbol Device:C
- added C4, C7: 100nF, Capacitor_SMD:C_0805_2012Metric, symbol Device:C
- added C5, C6: 1uF, Capacitor_SMD:C_0805_2012Metric, symbol Device:C
- added D1, D2, D3: LED, LED_SMD:LED_0805_2012Metric, symbol Device:LED
- added J5: Conn_01x02, Connector_PinHeader_2.54mm:PinHeader_1x02_P2.54mm_Vertical, symbol Connector_Generic:Conn_01x02
- J1, J4: footprint (none) -> Connector_PinHeader_2.54mm:PinHeader_1x08_P2.54mm_Vertical
- J2, J3: footprint (none) -> Connector_PinHeader_2.54mm:PinHeader_1x02_P2.54mm_Vertical
- R1, R10, R11, R2, R3, R4, R5, R6, R7, R8, R9: footprint (none) -> Resistor_SMD:R_0805_2012Metric
- RV1: footprint (none) -> Potentiometer_THT:Potentiometer_Bourns_3296W_Vertical
- U1, U2: footprint (none) -> Package_SO:MSOP-8_3x3mm_P0.65mm
Connections:
- net 15V: now also J2.2 (Pin_2), 1K3.2, C3.2, C4.2, C5.2; no longer J2.1 (Pin_1)
- net 3.3V: now also 1K2.1, C2.1
- net GND: now also J2.1 (Pin_1), C1.1, C2.2, C3.1, C4.1, C5.1, C6.2, C7.2, C8.2, D1.1 (K), D2.1 (K), D3.1 (K), J5.1 (Pin_1); no longer J2.2 (Pin_2)
- net L+: now also J4.1 (Pin_1)
- net M: now also J4.3 (Pin_3)
- net Q1: now also J4.4 (Pin_4)
- net Q2: now also J4.7 (Pin_7)
- net Vout: now also J4.8 (Pin_8), C6.1, C7.1, C8.1
- net 1.62V: now reaches U2.3 (+IN)
- net 1.62V: now also 1K1.2, C1.2, J5.2 (Pin_2)
- new net: 1K1.1, D1.2 (A)
- new net: 1K2.2, D2.2 (A)
- new net: 1K3.1, D3.2 (A)
- no-connect marks 0 -> 10
Other:
- moved on the sheet: J2, J3, J4
